File: PCB/floww.kicad_pcb (KiCad board)
At the start: 2 copper layers, 81.3 x 53.3 mm, 12 parts, among them J1 Conn_01x04_Male, J2 Conn_01x14_Male, SW1 SW_MEC_5E, SW2 SW_MEC_5E, SW3 SW_MEC_5E, SW4 SW_MEC_5E, U1 ATmega328P-P

Commit message: Add files via upload
Parts:
- moved R2 5.08 mm to (50.8, 91.4)
- moved C1 5.08 mm to (30.5, 55.9)
- moved J1 5.08 mm to (22.9, 61.0)
- moved SW3 5.08 mm to (25.4, 78.7)
- moved J2 5.08 mm to (91.4, 86.4)
- moved R1 5.08 mm to (35.6, 91.4)
- moved R3 5.08 mm to (20.3, 91.4)
- moved REF** 5.08 mm to (81.3, 91.4)
- moved SW1 5.08 mm to (40.6, 78.7)
- moved SW2 5.08 mm to (55.9, 78.7)
- moved SW4 5.08 mm to (71.1, 78.7)
- moved U1 5.08 mm to (72.4, 54.6)
Other:
- board text added: "Made in FabLab - Mérida"
